Commit message: Fixed interface loading

File: chudovishe_description/urdf/chudovishe_base.urdf.xacro (robot description, xacro)
@@ -119,4 +119,23 @@
     <origin xyz="-0.12 0 -0.0125" rpy="0 0 0"/>
   </joint>
-<xacro:chudovishe_ros2_control/>
+<ros2_control name="ArduinoDiffDrive" type="system">
+  <hardware>
+    <plugin>chudovishe_hardware/DiffDriveArduinoHardware</plugin>
+    <param name="device">/dev/ttyACM0</param>
+    <param name="baud_rate">57600</param>
+    <param name="timeout_ms">5</param>
+    <param name="enc_counts_per_rev">1123</param>
+    <param name="reset_encoders_on_activate">true</param>
+  </hardware>
+  <joint name="left_wheel_joint">
+    <command_interface name="velocity"/>
+    <state_interface name="position"/>
+    <state_interface name="velocity"/>
+  </joint>
+  <joint name="right_wheel_joint">
+    <command_interface name="velocity"/>
+    <state_interface name="position"/>
+    <state_interface name="velocity"/>
+  </joint>
+</ros2_control>
 </robot>

Commit message: Hardware rewrite

File: chudovishe_description/urdf/chudovishe_base.urdf.xacro (robot description, xacro)
@@ -119,12 +119,12 @@
     <origin xyz="-0.12 0 -0.0125" rpy="0 0 0"/>
   </joint>
-<ros2_control name="ArduinoDiffDrive" type="system">
+<ros2_control name="ChudovisheSystemHardware" type="system">
   <hardware>
-    <plugin>chudovishe_hardware/DiffDriveArduinoHardware</plugin>
-    <param name="device">/dev/ttyACM0</param>
-    <param name="baud_rate">57600</param>
-    <param name="timeout_ms">5</param>
+    <plugin>chudovishe_hardware/ChudovisheSystemHardware</plugin>
+    <param name="port_name">/dev/ttyACM0</param>
+    <param name="baudrate">57600</param>
+    <!-- <param name="timeout_ms">50</param>
     <param name="enc_counts_per_rev">1123</param>
-    <param name="reset_encoders_on_activate">true</param>
+    <param name="reset_encoders_on_activate">true</param> -->
   </hardware>
   <joint name="left_wheel_joint">

File: chudovishe_description/urdf/ros2_control.urdf.xacro (robot description, xacro)
@@ -1,13 +1,12 @@
 <?xml version="1.0"?>
 <robot xmlns:xacro="http://www.ros.org/wiki/xacro">
-  <xacro:macro name="chudovishe_ros2_control">
 <ros2_control name="ArduinoDiffDrive" type="system">
   <hardware>
-    <plugin>chudovishe_hardware/DiffDriveArduinoHardware</plugin>
-    <param name="device">/dev/ttyACM0</param>
-    <param name="baud_rate">57600</param>
-    <param name="timeout_ms">50</param>
+    <plugin>chudovishe_hardware/ChudovisheSystemHardware</plugin>
+    <param name="port_name">/dev/ttyACM0</param>
+    <param name="baudrate">57600</param>
+    <!-- <param name="timeout_ms">50</param>
     <param name="enc_counts_per_rev">1123</param>
-    <param name="reset_encoders_on_activate">true</param>
+    <param name="reset_encoders_on_activate">true</param> -->
   </hardware>
   <joint name="left_wheel_joint">
@@ -22,4 +21,3 @@
   </joint>
 </ros2_control>
-  </xacro:macro>
 </robot>
